File: single_esc.sch (KiCad schematic (older format))
At the start: 21 parts, among them U501 EFM8BB21

Commit message: kicad-upgrade to v6
Parts:
- BL_TX1, OUT_A501, OUT_B501, OUT_C501, TP502: symbol TP -> custom:TP
- C501, C502: symbol CUSTOM_C -> custom:CUSTOM_C
- FET501, FET503, FET505: symbol IRLML6244 -> custom:IRLML6244
- FET502, FET504, FET506: symbol IRLML2244 -> custom:IRLML2244
- R501, R502, R503, R504, R505, R506, R507: symbol CUSTOM_R -> custom:CUSTOM_R
- U501: symbol EFM8BB21 -> custom:EFM8BB21
Connections:
- wire segments 79 -> 99
