File: tinyPEPPER.sch (KiCad schematic (older format))
At the start: 11 parts

Commit message: kicad-upgrade to v6
Parts:
- C1000: symbol CUSTOM_C -> custom:CUSTOM_C
- H1, H2, H3, H4: symbol hole -> custom:hole
- TP101, TP102, TP103, TP104, TP105, TP106: symbol TP -> custom:TP
Connections:
- wire segments 26 -> 34
Changed lines of the file:
@@
-EESchema Schematic File Version 2
-LIBS:power
-LIBS:device
-LIBS:transistors
-LIBS:conn
-LIBS:linear
-LIBS:regul
-LIBS:74xx
-LIBS:cmos4000
-LIBS:adc-dac
-LIBS:memory
-LIBS:xilinx
-LIBS:microcontrollers
-LIBS:dsp
-LIBS:microchip
-LIBS:analog_switches
-LIBS:motorola
-LIBS:texas
-LIBS:intel
-LIBS:audio
-LIBS:interface
-LIBS:digital-audio
-LIBS:philips
-LIBS:display
-LIBS:cypress
-LIBS:siliconi
-LIBS:opto
-LIBS:atmel
-LIBS:contrib
-LIBS:valves
-LIBS:custom
-LIBS:tinyPEPPER-cache
-EELAYER 26 0
+EESchema Schematic File Version 4
+EELAYER 30 0
 EELAYER END
 $Descr A4 11693 8268
@@
 $EndDescr
 $Comp
-L TP TP101
+L custom:TP TP101
 U 1 1 57F7AE6B
 P 1600 2450
@@
 $EndComp
 $Comp
-L TP TP102
+L custom:TP TP102
 U 1 1 57F7AE9E
 P 1600 2700
@@
 $EndComp
 $Comp
-L TP TP103
+L custom:TP TP103
 U 1 1 57F7AEE5
 P 1600 3350
@@
 $EndComp
 $Comp
-L TP TP104
+L custom:TP TP104
 U 1 1 57F7AEF4
 P 1600 3600
@@
 $EndComp
 $Comp
-L TP TP105
+L custom:TP TP105
 U 1 1 57F7AF0C
 P 1600 3850
@@
 $EndComp
 $Comp
-L TP TP106
+L custom:TP TP106
 U 1 1 57F7AF1B
 P 1600 4150
@@
 $EndComp
 Wire Wire Line
-	1900 2450 4700 2450
-Wire Wire Line
-	1900 2700 4700 2700
+	1900 2450 2600 2450
+Wire Wire Line
+	1900 2700 3000 2700
 Wire Wire Line
 	1900 3350 2900 3350
@@
 	4450 3900 4700 3900
 Wire Wire Line
-	4450 2700 4450 6150
+	4450 2700 4450 3900
 Connection ~ 4450 2700
 Wire Wire Line
-	4600 2450 4600 5950
+	4600 2450 4600 3700
 Wire Wire Line
 	4600 3700 4700 3700
@@
 Connection ~ 4600 4800
 $Comp
-L CUSTOM_C C1000
+L custom:CUSTOM_C C1000
 U 1 1 57FCB86E
 P 2800 2250
@@
 Connection ~ 3000 2700
 $Comp
-L hole H1
+L custom:hole H1
 U 1 1 58465F4C
 P 9500 2250
@@
 $EndComp
 $Comp
-L hole H2
+L custom:hole H2
 U 1 1 58466048
 P 9500 2700
@@
 $EndComp
 $Comp
-L hole H3
+L custom:hole H3
 U 1 1 58466181
 P 10200 2250
@@
 $EndComp
 $Comp
-L hole H4
+L custom:hole H4
 U 1 1 58466291
 P 10200 2700
@@
 Wire Wire Line
 	2950 2250 3000 2250
+Wire Wire Line
+	4450 2700 4700 2700
+Wire Wire Line
+	4600 2450 4700 2450
+Wire Wire Line
+	4450 3900 4450 5000
+Wire Wire Line
+	4450 5000 4450 6150
+Wire Wire Line
+	4600 3700 4600 4800
+Wire Wire Line
+	4600 4800 4600 5950
+Wire Wire Line
+	2600 2450 4600 2450
+Wire Wire Line
+	3000 2700 4450 2700
 $EndSCHEMATC
