File: power.kicad_sch (KiCad schematic)
At the start: 6 parts

Commit message: added 3v3-reg
Parts:
- added C? (x2): 1uF, symbol pspice:C
- added D?: DIODE, symbol pspice:DIODE
- added U?: RT9013-33GB, SOT94P279X129-5N, symbol RT9013-33GB:RT9013-33GB
Connections:
- net 3.3V: now also C?.1, U?.5 (VOUT)
- net 5V: now also C?.1, D?.2 (A), U?.1 (VIN), U?.3 (EN)
- net GND: now also C?.2, U?.2 (GND)
- new net VBUS: D?.1 (K)
Changed lines of the file:
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@@
 (kicad_sch (version 20211123) (generator eeschema)
   (paper "A4")
+  (junction (at 93.98 129.54) (diameter 0) (color 0 0 0 0)
+  )
+  (junction (at 113.03 129.54) (diameter 0) (color 0 0 0 0)
+  )
   (junction (at 115.57 86.36) (diameter 0) (color 0 0 0 0)
   )
@@
   (junction (at 97.79 52.07) (diameter 0) (color 0 0 0 0)
   )
+  (junction (at 80.01 110.49) (diameter 0) (color 0 0 0 0)
+  )
+  (junction (at 76.2 105.41) (diameter 0) (color 0 0 0 0)
+  )
   (junction (at 198.12 73.66) (diameter 0) (color 0 0 0 0)
   )
@@
   (junction (at 115.57 71.12) (diameter 0) (color 0 0 0 0)
   )
+  (wire (pts (xy 113.03 129.54) (xy 113.03 133.35))
+    (stroke (width 0) (type default) (color 0 0 0 0))
+  )
   (wire (pts (xy 107.95 76.2) (xy 107.95 45.72))
     (stroke (width 0) (type default) (color 0 0 0 0))
@@
     (stroke (width 0) (type default) (color 0 0 0 0))
   )
+  (wire (pts (xy 43.18 110.49) (xy 43.18 90.17))
+    (stroke (width 0) (type default) (color 0 0 0 0))
+  )
+  (wire (pts (xy 76.2 105.41) (xy 93.98 105.41))
+    (stroke (width 0) (type default) (color 0 0 0 0))
+  )
   (wire (pts (xy 151.13 71.12) (xy 151.13 73.66))
     (stroke (width 0) (type default) (color 0 0 0 0))
@@
     (stroke (width 0) (type default) (color 0 0 0 0))
   )
+  (wire (pts (xy 80.01 110.49) (xy 80.01 116.84))
+    (stroke (width 0) (type default) (color 0 0 0 0))
+  )
   (wire (pts (xy 97.79 52.07) (xy 115.57 52.07))
     (stroke (width 0) (type default) (color 0 0 0 0))
   )
+  (wire (pts (xy 93.98 142.24) (xy 93.98 146.05))
+    (stroke (width 0) (type default) (color 0 0 0 0))
+  )
+  (wire (pts (xy 93.98 105.41) (xy 93.98 129.54))
+    (stroke (width 0) (type default) (color 0 0 0 0))
+  )
   (wire (pts (xy 86.36 81.28) (xy 115.57 81.28))
     (stroke (width 0) (type default) (color 0 0 0 0))
   )
+  (wire (pts (xy 113.03 129.54) (xy 198.12 129.54))
+    (stroke (width 0) (type default) (color 0 0 0 0))
+  )
+  (wire (pts (xy 76.2 90.17) (xy 76.2 105.41))
+    (stroke (width 0) (type default) (color 0 0 0 0))
+  )
   (wire (pts (xy 113.03 78.74) (xy 115.57 78.74))
     (stroke (width 0) (type default) (color 0 0 0 0))
@@
     (stroke (width 0) (type default) (color 0 0 0 0))
   )
+  (wire (pts (xy 93.98 129.54) (xy 113.03 129.54))
+    (stroke (width 0) (type default) (color 0 0 0 0))
+  )
   (wire (pts (xy 113.03 106.68) (xy 113.03 111.76))
     (stroke (width 0) (type default) (color 0 0 0 0))
@@
     (stroke (width 0) (type default) (color 0 0 0 0))
   )
+  (wire (pts (xy 43.18 90.17) (xy 76.2 90.17))
+    (stroke (width 0) (type default) (color 0 0 0 0))
+  )
+  (wire (pts (xy 73.66 110.49) (xy 80.01 110.49))
+    (stroke (width 0) (type default) (color 0 0 0 0))
+  )
   (wire (pts (xy 110.49 86.36) (xy 115.57 86.36))
     (stroke (width 0) (type default) (color 0 0 0 0))
@@
     (stroke (width 0) (type default) (color 0 0 0 0))
   )
+  (wire (pts (xy 73.66 105.41) (xy 76.2 105.41))
+    (stroke (width 0) (type default) (color 0 0 0 0))
+  )
+  (wire (pts (xy 113.03 143.51) (xy 113.03 151.13))
+    (stroke (width 0) (type default) (color 0 0 0 0))
+  )
   (wire (pts (xy 115.57 52.07) (xy 115.57 71.12))
     (stroke (width 0) (type default) (color 0 0 0 0))
@@
     (stroke (width 0) (type default) (color 0 0 0 0))
   )
+  (wire (pts (xy 80.01 110.49) (xy 83.82 110.49))
+    (stroke (width 0) (type default) (color 0 0 0 0))
+  )
   (wire (pts (xy 78.74 64.77) (xy 78.74 69.85))
     (stroke (width 0) (type default) (color 0 0 0 0))
   )
+  (wire (pts (xy 73.66 115.57) (xy 73.66 127))
+    (stroke (width 0) (type default) (color 0 0 0 0))
+  )
   (wire (pts (xy 66.04 52.07) (xy 78.74 52.07))
     (stroke (width 0) (type default) (color 0 0 0 0))
@@
     (stroke (width 0) (type default) (color 0 0 0 0))
   )
+  (wire (pts (xy 198.12 129.54) (xy 198.12 73.66))
+    (stroke (width 0) (type default) (color 0 0 0 0))
+  )
   (hierarchical_label "GND" (shape input) (at 86.36 81.28 180)
     (effects (font (size 1.524 1.524)) (justify right))
@@
     (effects (font (size 1.524 1.524)) (justify right))
   )
+  (hierarchical_label "GND" (shape input) (at 73.66 127 270)
+    (effects (font (size 1.524 1.524)) (justify right))
+  )
+  (hierarchical_label "GND" (shape input) (at 93.98 146.05 270)
+    (effects (font (size 1.524 1.524)) (justify right))
+  )
   (hierarchical_label "GND" (shape input) (at 113.03 111.76 270)
     (effects (font (size 1.524 1.524)) (justify right))
   )
-  (hierarchical_label "3.3V" (shape output) (at 34.29 74.93 180)
-    (effects (font (size 1.524 1.524)) (justify right))
+  (hierarchical_label "VBUS" (shape input) (at 113.03 151.13 270)
+    (effects (font (size 1.524 1.524)) (justify right))
+  )
+  (hierarchical_label "3.3V" (shape output) (at 83.82 110.49 0)
+    (effects (font (size 1.524 1.524)) (justify left))
   )
   (hierarchical_label "5V" (shape output) (at 203.2 73.66 0)
@@
     (pin "2")
   )
+  (symbol (lib_id "RT9013-33GB:RT9013-33GB") (at 58.42 110.49 0) (unit 1)
+    (in_bom yes) (on_board yes) (fields_autoplaced)
+    (property "Reference" "U?" (id 0) (at 58.42 97.79 0))
+    (property "Value" "RT9013-33GB" (id 1) (at 58.42 100.33 0))
+    (property "Footprint" "SOT94P279X129-5N" (id 2) (at 58.42 110.49 0)
+      (effects (font (size 1.27 1.27)) (justify bottom) hide)
+    )
+    (property "Datasheet" "" (id 3) (at 58.42 110.49 0)
+      (effects (font (size 1.27 1.27)) hide)
+    )
+    (property "MANUFACTURER" "Richtek Technology" (id 4) (at 58.42 110.49 0)
+      (effects (font (size 1.27 1.27)) (justify bottom) hide)
+    )
+    (property "PARTREV" "Aprill 2011" (id 5) (at 58.42 110.49 0)
+      (effects (font (size 1.27 1.27)) (justify bottom) hide)
+    )
+    (property "MAXIMUM_PACKAGE_HEIGHT" "1.295 mm" (id 6) (at 58.42 110.49 0)
+      (effects (font (size 1.27 1.27)) (justify bottom) hide)
+    )
+    (property "STANDARD" "IPC 7351B" (id 7) (at 58.42 110.49 0)
+      (effects (font (size 1.27 1.27)) (justify bottom) hide)
+    )
+    (pin "1")
+    (pin "2")
+    (pin "3")
+    (pin "5")
+  )
+  (symbol (lib_id "pspice:C") (at 93.98 135.89 0) (unit 1)
+    (in_bom yes) (on_board yes) (fields_autoplaced)
+    (property "Reference" "C?" (id 0) (at 99.06 134.6199 0)
+      (effects (font (size 1.27 1.27)) (justify left))
+    )
+    (property "Value" "1uF" (id 1) (at 99.06 137.1599 0)
+      (effects (font (size 1.27 1.27)) (justify left))
+    )
+    (property "Footprint" "" (id 2) (at 93.98 135.89 0)
+      (effects (font (size 1.27 1.27)) hide)
+    )
+    (property "Datasheet" "~" (id 3) (at 93.98 135.89 0)
+      (effects (font (size 1.27 1.27)) hide)
+    )
+    (pin "1")
+    (pin "2")
+  )
   (symbol (lib_id "pspice:C") (at 78.74 58.42 0) (unit 1)
     (in_bom yes) (on_board yes) (fields_autoplaced)
@@
     )
     (property "Datasheet" "~" (id 3) (at 168.91 80.01 0)
+      (effects (font (size 1.27 1.27)) hide)
+    )
+    (pin "1")
+    (pin "2")
+  )
+  (symbol (lib_id "pspice:DIODE") (at 113.03 138.43 90) (unit 1)
+    (in_bom yes) (on_board yes) (fields_autoplaced)
+    (property "Reference" "D?" (id 0) (at 116.84 137.1599 90)
+      (effects (font (size 1.27 1.27)) (justify right))
+    )
+    (property "Value" "DIODE" (id 1) (at 116.84 139.6999 90)
+      (effects (font (size 1.27 1.27)) (justify right))
+    )
+    (property "Footprint" "" (id 2) (at 113.03 138.43 0)
+      (effects (font (size 1.27 1.27)) hide)
+    )
+    (property "Datasheet" "~" (id 3) (at 113.03 138.43 0)
       (effects (font (size 1.27 1.27)) hide)
     )
@@
     (pin "9")
   )
+  (symbol (lib_id "pspice:C") (at 80.01 123.19 0) (unit 1)
+    (in_bom yes) (on_board yes) (fields_autoplaced)
+    (property "Reference" "C?" (id 0) (at 85.09 121.9199 0)
+      (effects (font (size 1.27 1.27)) (justify left))
+    )
+    (property "Value" "1uF" (id 1) (at 85.09 124.4599 0)
+      (effects (font (size 1.27 1.27)) (justify left))
+    )
+    (property "Footprint" "" (id 2) (at 80.01 123.19 0)
+      (effects (font (size 1.27 1.27)) hide)
+    )
+    (property "Datasheet" "~" (id 3) (at 80.01 123.19 0)
+      (effects (font (size 1.27 1.27)) hide)
+    )
+    (pin "1")
+    (pin "2")
+  )
 )
