File: mcu.kicad_sch (KiCad schematic)
At the start: 1 part

Commit message: added further parts
Parts:
- added J?: Micro_SD_Card, symbol Connector:Micro_SD_Card
- added P?: USB_C_Plug, symbol Connector:USB_C_Plug
- added U?: ICM-20602, Package_LGA:LGA-16_3x3mm_P0.5mm_LayoutBorder3x5y, symbol Sensor_Motion:ICM-20602
- added U?: BMP280, Package_LGA:Bosch_LGA-8_2x2.5mm_P0.65mm_ClockwisePinNumbering, symbol Sensor_Pressure:BMP280
Connections:
- new net: U?.10 (GND), U?.11 (GND), U?.12 (GND), U?.13 (GND), U?.15 (GND), U?.9 (GND)
- new net: P?.A1 (GND), P?.A12 (GND), P?.B1 (GND), P?.B12 (GND)
- new net: P?.A4 (VBUS), P?.A9 (VBUS), P?.B4 (VBUS), P?.B9 (VBUS)
Changed lines of the file:
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@@
 (kicad_sch (version 20211123) (generator eeschema)
   (paper "A4")
+  (hierarchical_label "TELEM_TX" (shape output) (at 43.18 154.94 180)
+    (effects (font (size 1.524 1.524)) (justify right))
+  )
+  (hierarchical_label "TELEM_RX" (shape input) (at 43.18 158.75 180)
+    (effects (font (size 1.524 1.524)) (justify right))
+  )
+  (hierarchical_label "GPS_TX" (shape output) (at 44.45 138.43 180)
+    (effects (font (size 1.524 1.524)) (justify right))
+  )
+  (hierarchical_label "GPS_RX" (shape input) (at 44.45 142.24 180)
+    (effects (font (size 1.524 1.524)) (justify right))
+  )
+  (hierarchical_label "GND" (shape input) (at 53.34 50.8 180)
+    (effects (font (size 1.524 1.524)) (justify right))
+  )
   (hierarchical_label "MOTOR 1" (shape output) (at 45.72 86.36 180)
     (effects (font (size 1.524 1.524)) (justify right))
   )
+  (hierarchical_label "RC_RX" (shape input) (at 45.72 127 180)
+    (effects (font (size 1.524 1.524)) (justify right))
+  )
   (hierarchical_label "3.3V" (shape input) (at 53.34 45.72 180)
     (effects (font (size 1.524 1.524)) (justify right))
@@
     (effects (font (size 1.524 1.524)) (justify right))
   )
+  (hierarchical_label "RC_TX" (shape output) (at 45.72 123.19 180)
+    (effects (font (size 1.524 1.524)) (justify right))
+  )
   (hierarchical_label "MOTOR 2" (shape output) (at 45.72 92.71 180)
     (effects (font (size 1.524 1.524)) (justify right))
@@
   (hierarchical_label "MOTOR 3" (shape output) (at 45.72 99.06 180)
     (effects (font (size 1.524 1.524)) (justify right))
+  )
+  (symbol (lib_id "Sensor_Motion:ICM-20602") (at 170.18 46.99 0) (unit 1)
+    (in_bom yes) (on_board yes) (fields_autoplaced)
+    (property "Reference" "U?" (id 0) (at 172.1994 59.69 0)
+      (effects (font (size 1.27 1.27)) (justify left))
+    )
+    (property "Value" "ICM-20602" (id 1) (at 172.1994 62.23 0)
+      (effects (font (size 1.27 1.27)) (justify left))
+    )
+    (property "Footprint" "Package_LGA:LGA-16_3x3mm_P0.5mm_LayoutBorder3x5y" (id 2) (at 170.18 40.64 0)
+      (effects (font (size 1.27 1.27)) hide)
+    )
+    (property "Datasheet" "http://www.invensense.com/wp-content/uploads/2016/10/DS-000176-ICM-20602-v1.0.pdf" (id 3) (at 171.45 22.86 0)
+      (effects (font (size 1.27 1.27)) hide)
+    )
+    (pin "1")
+    (pin "10")
+    (pin "11")
+    (pin "12")
+    (pin "13")
+    (pin "14")
+    (pin "15")
+    (pin "16")
+    (pin "2")
+    (pin "3")
+    (pin "4")
+    (pin "5")
+    (pin "6")
+    (pin "7")
+    (pin "8")
+    (pin "9")
+  )
+  (symbol (lib_id "Sensor_Pressure:BMP280") (at 167.64 139.7 0) (unit 1)
+    (in_bom yes) (on_board yes) (fields_autoplaced)
+    (property "Reference" "U?" (id 0) (at 173.99 137.1599 0)
+      (effects (font (size 1.27 1.27)) (justify left))
+    )
+    (property "Value" "BMP280" (id 1) (at 173.99 139.6999 0)
+      (effects (font (size 1.27 1.27)) (justify left))
+    )
+    (property "Footprint" "Package_LGA:Bosch_LGA-8_2x2.5mm_P0.65mm_ClockwisePinNumbering" (id 2) (at 167.64 157.48 0)
+      (effects (font (size 1.27 1.27)) hide)
+    )
+    (property "Datasheet" "https://ae-bst.resource.bosch.com/media/_tech/media/datasheets/BST-BMP280-DS001.pdf" (id 3) (at 167.64 139.7 0)
+      (effects (font (size 1.27 1.27)) hide)
+    )
+    (pin "1")
+    (pin "2")
+    (pin "3")
+    (pin "4")
+    (pin "5")
+    (pin "6")
+    (pin "7")
+    (pin "8")
   )
   (symbol (lib_id "MCU_ST_STM32F4:STM32F405RGTx") (at 105.41 92.71 0) (unit 1)
@@
     (pin "9")
   )
+  (symbol (lib_id "Connector:Micro_SD_Card") (at 193.04 92.71 0) (unit 1)
+    (in_bom yes) (on_board yes) (fields_autoplaced)
+    (property "Reference" "J?" (id 0) (at 193.675 73.66 0))
+    (property "Value" "Micro_SD_Card" (id 1) (at 193.675 76.2 0))
+    (property "Footprint" "" (id 2) (at 222.25 85.09 0)
+      (effects (font (size 1.27 1.27)) hide)
+    )
+    (property "Datasheet" "http://katalog.we-online.de/em/datasheet/693072010801.pdf" (id 3) (at 193.04 92.71 0)
+      (effects (font (size 1.27 1.27)) hide)
+    )
+    (pin "1")
+    (pin "2")
+    (pin "3")
+    (pin "4")
+    (pin "5")
+    (pin "6")
+    (pin "7")
+    (pin "8")
+    (pin "9")
+  )
+  (symbol (lib_id "Connector:USB_C_Plug") (at 248.92 77.47 0) (unit 1)
+    (in_bom yes) (on_board yes) (fields_autoplaced)
+    (property "Reference" "P?" (id 0) (at 248.92 44.45 0))
+    (property "Value" "USB_C_Plug" (id 1) (at 248.92 46.99 0))
+    (property "Footprint" "" (id 2) (at 252.73 77.47 0)
+      (effects (font (size 1.27 1.27)) hide)
+    )
+    (property "Datasheet" "https://www.usb.org/sites/default/files/documents/usb_type-c.zip" (id 3) (at 252.73 77.47 0)
+      (effects (font (size 1.27 1.27)) hide)
+    )
+    (pin "A1")
+    (pin "A10")
+    (pin "A11")
+    (pin "A12")
+    (pin "A2")
+    (pin "A3")
+    (pin "A4")
+    (pin "A5")
+    (pin "A6")
+    (pin "A7")
+    (pin "A8")
+    (pin "A9")
+    (pin "B1")
+    (pin "B10")
+    (pin "B11")
+    (pin "B12")
+    (pin "B2")
+    (pin "B3")
+    (pin "B4")
+    (pin "B5")
+    (pin "B8")
+    (pin "B9")
+    (pin "S1")
+  )
 )

Commit message: added correct usb plug
Parts:
- removed P?: USB_C_Plug, symbol Connector:USB_C_Plug
- added J?: TYPE-C-31-M-12, HRO_TYPE-C-31-M-12, symbol TYPE-C-31-M-12:TYPE-C-31-M-12
Connections:
- net GND: now also U?.18 (VSS), U?.63 (VSS)
- net MOTOR 1: now also U?.26 (PB0)
- net MOTOR 2: now also U?.27 (PB1)
- net MOTOR 3: now also U?.17 (PA3)
- net MOTOR 4: now also U?.16 (PA2)
- net D-: now reaches U?.44 (PA11)
- net D-: now also J?.A7 (DN1)
- net D+: now reaches U?.45 (PA12)
- net D+: now also J?.A6 (DP1)
- net BOOT0: now reaches U?.60 (BOOT0)
- new net: J?.A1_B12 (GND), J?.B1_A12 (GND)
- new net: J?.A4_B9 (VBUS), J?.B4_A9 (VBUS)
- new net: J?.S1 (SHIELD), J?.S2 (SHIELD), J?.S3 (SHIELD), J?.S4 (SHIELD)
Other:
- moved on the sheet: U?
Changed lines of the file:
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@@
 (kicad_sch (version 20211123) (generator eeschema)
   (paper "A4")
+  (junction (at 102.87 142.24) (diameter 0) (color 0 0 0 0)
+  )
+  (wire (pts (xy 102.87 138.43) (xy 102.87 142.24))
+    (stroke (width 0) (type default) (color 0 0 0 0))
+  )
+  (wire (pts (xy 102.87 142.24) (xy 102.87 146.05))
+    (stroke (width 0) (type default) (color 0 0 0 0))
+  )
+  (wire (pts (xy 100.33 138.43) (xy 100.33 142.24))
+    (stroke (width 0) (type default) (color 0 0 0 0))
+  )
+  (wire (pts (xy 120.65 80.01) (xy 127 80.01))
+    (stroke (width 0) (type default) (color 0 0 0 0))
+  )
+  (wire (pts (xy 100.33 142.24) (xy 102.87 142.24))
+    (stroke (width 0) (type default) (color 0 0 0 0))
+  )
+  (wire (pts (xy 120.65 57.15) (xy 125.73 57.15))
+    (stroke (width 0) (type default) (color 0 0 0 0))
+  )
+  (wire (pts (xy 120.65 97.79) (xy 125.73 97.79))
+    (stroke (width 0) (type default) (color 0 0 0 0))
+  )
+  (wire (pts (xy 120.65 59.69) (xy 125.73 59.69))
+    (stroke (width 0) (type default) (color 0 0 0 0))
+  )
+  (wire (pts (xy 120.65 82.55) (xy 127 82.55))
+    (stroke (width 0) (type default) (color 0 0 0 0))
+  )
+  (wire (pts (xy 120.65 95.25) (xy 125.73 95.25))
+    (stroke (width 0) (type default) (color 0 0 0 0))
+  )
+  (wire (pts (xy 76.2 57.15) (xy 85.09 57.15))
+    (stroke (width 0) (type default) (color 0 0 0 0))
+  )
+  (wire (pts (xy 207.01 139.7) (xy 212.09 139.7))
+    (stroke (width 0) (type default) (color 0 0 0 0))
+  )
+  (wire (pts (xy 207.01 142.24) (xy 212.09 142.24))
+    (stroke (width 0) (type default) (color 0 0 0 0))
+  )
+  (label "D+" (at 207.01 139.7 180)
+    (effects (font (size 1.524 1.524)) (justify right bottom))
+  )
+  (label "D-" (at 207.01 142.24 180)
+    (effects (font (size 1.524 1.524)) (justify right bottom))
+  )
+  (label "D+" (at 127 82.55 0)
+    (effects (font (size 1.524 1.524)) (justify left bottom))
+  )
+  (label "D-" (at 127 80.01 0)
+    (effects (font (size 1.524 1.524)) (justify left bottom))
+  )
+  (label "BOOT0" (at 76.2 57.15 180)
+    (effects (font (size 1.524 1.524)) (justify right bottom))
+  )
   (hierarchical_label "TELEM_TX" (shape output) (at 43.18 154.94 180)
     (effects (font (size 1.524 1.524)) (justify right))
   )
+  (hierarchical_label "MOTOR 2" (shape output) (at 125.73 97.79 0)
+    (effects (font (size 1.524 1.524)) (justify left))
+  )
   (hierarchical_label "TELEM_RX" (shape input) (at 43.18 158.75 180)
     (effects (font (size 1.524 1.524)) (justify right))
@@
     (effects (font (size 1.524 1.524)) (justify right))
   )
-  (hierarchical_label "GND" (shape input) (at 53.34 50.8 180)
-    (effects (font (size 1.524 1.524)) (justify right))
-  )
-  (hierarchical_label "MOTOR 1" (shape output) (at 45.72 86.36 180)
-    (effects (font (size 1.524 1.524)) (justify right))
+  (hierarchical_label "GND" (shape input) (at 102.87 146.05 270)
+    (effects (font (size 1.524 1.524)) (justify right))
+  )
+  (hierarchical_label "MOTOR 1" (shape output) (at 125.73 95.25 0)
+    (effects (font (size 1.524 1.524)) (justify left))
   )
   (hierarchical_label "RC_RX" (shape input) (at 45.72 127 180)
     (effects (font (size 1.524 1.524)) (justify right))
   )
+  (hierarchical_label "LED" (shape output) (at 36.83 166.37 180)
+    (effects (font (size 1.524 1.524)) (justify right))
+  )
   (hierarchical_label "3.3V" (shape input) (at 53.34 45.72 180)
     (effects (font (size 1.524 1.524)) (justify right))
   )
-  (hierarchical_label "MOTOR 4" (shape output) (at 45.72 105.41 180)
-    (effects (font (size 1.524 1.524)) (justify right))
+  (hierarchical_label "MOTOR 4" (shape output) (at 125.73 57.15 0)
+    (effects (font (size 1.524 1.524)) (justify left))
   )
   (hierarchical_label "RC_TX" (shape output) (at 45.72 123.19 180)
     (effects (font (size 1.524 1.524)) (justify right))
   )
-  (hierarchical_label "MOTOR 2" (shape output) (at 45.72 92.71 180)
-    (effects (font (size 1.524 1.524)) (justify right))
-  )
-  (hierarchical_label "MOTOR 3" (shape output) (at 45.72 99.06 180)
-    (effects (font (size 1.524 1.524)) (justify right))
+  (hierarchical_label "MOTOR 3" (shape output) (at 125.73 59.69 0)
+    (effects (font (size 1.524 1.524)) (justify left))
   )
   (symbol (lib_id "Sensor_Motion:ICM-20602") (at 170.18 46.99 0) (unit 1)
@@
     (pin "8")
   )
-  (symbol (lib_id "MCU_ST_STM32F4:STM32F405RGTx") (at 105.41 92.71 0) (unit 1)
-    (in_bom yes) (on_board yes) (fields_autoplaced)
-    (property "Reference" "U?" (id 0) (at 109.9694 138.43 0)
-      (effects (font (size 1.27 1.27)) (justify left))
-    )
-    (property "Value" "STM32F405RGTx" (id 1) (at 109.9694 140.97 0)
-      (effects (font (size 1.27 1.27)) (justify left))
-    )
-    (property "Footprint" "Package_QFP:LQFP-64_10x10mm_P0.5mm" (id 2) (at 90.17 135.89 0)
+  (symbol (lib_id "TYPE-C-31-M-12:TYPE-C-31-M-12") (at 229.87 142.24 0) (unit 1)
+    (in_bom yes) (on_board yes) (fields_autoplaced)
+    (property "Reference" "J?" (id 0) (at 229.87 124.46 0))
+    (property "Value" "TYPE-C-31-M-12" (id 1) (at 229.87 127 0))
+    (property "Footprint" "HRO_TYPE-C-31-M-12" (id 2) (at 229.87 142.24 0)
+      (effects (font (size 1.27 1.27)) (justify bottom) hide)
+    )
+    (property "Datasheet" "" (id 3) (at 229.87 142.24 0)
+      (effects (font (size 1.27 1.27)) hide)
+    )
+    (property "STANDARD" "Manufacturer Recommendations" (id 4) (at 229.87 142.24 0)
+      (effects (font (size 1.27 1.27)) (justify bottom) hide)
+    )
+    (property "SNAPEDA_PN" "TYPE-C-31-M-12" (id 5) (at 229.87 142.24 0)
+      (effects (font (size 1.27 1.27)) (justify bottom) hide)
+    )
+    (property "PARTREV" "2020.12.08" (id 6) (at 229.87 142.24 0)
+      (effects (font (size 1.27 1.27)) (justify bottom) hide)
+    )
+    (property "MANUFACTURER" "HRO Electronics Co., Ltd." (id 7) (at 229.87 142.24 0)
+      (effects (font (size 1.27 1.27)) (justify bottom) hide)
+    )
+    (property "MAXIMUM_PACKAGE_HEIGHT" "3.26 mm" (id 8) (at 229.87 142.24 0)
+      (effects (font (size 1.27 1.27)) (justify bottom) hide)
+    )
+    (pin "A1_B12")
+    (pin "A4_B9")
+    (pin "A5")
+    (pin "A6")
+    (pin "A7")
+    (pin "A8")
+    (pin "B1_A12")
+    (pin "B4_A9")
+    (pin "B5")
+    (pin "B6")
+    (pin "B7")
+    (pin "B8")
+    (pin "S1")
+    (pin "S2")
+    (pin "S3")
+    (pin "S4")
+  )
+  (symbol (lib_id "MCU_ST_STM32F4:STM32F405RGTx") (at 102.87 92.71 0) (unit 1)
+    (in_bom yes) (on_board yes) (fields_autoplaced)
+    (property "Reference" "U?" (id 0) (at 107.4294 138.43 0)
+      (effects (font (size 1.27 1.27)) (justify left))
+    )
+    (property "Value" "STM32F405RGTx" (id 1) (at 107.4294 140.97 0)
+      (effects (font (size 1.27 1.27)) (justify left))
+    )
+    (property "Footprint" "Package_QFP:LQFP-64_10x10mm_P0.5mm" (id 2) (at 87.63 135.89 0)
       (effects (font (size 1.27 1.27)) (justify right) hide)
     )
-    (property "Datasheet" "http://www.st.com/st-web-ui/static/active/en/resource/technical/document/datasheet/DM00037051.pdf" (id 3) (at 105.41 92.71 0)
+    (property "Datasheet" "http://www.st.com/st-web-ui/static/active/en/resource/technical/document/datasheet/DM00037051.pdf" (id 3) (at 102.87 92.71 0)
       (effects (font (size 1.27 1.27)) hide)
     )
@@
     (pin "9")
   )
-  (symbol (lib_id "Connector:USB_C_Plug") (at 248.92 77.47 0) (unit 1)
-    (in_bom yes) (on_board yes) (fields_autoplaced)
-    (property "Reference" "P?" (id 0) (at 248.92 44.45 0))
-    (property "Value" "USB_C_Plug" (id 1) (at 248.92 46.99 0))
-    (property "Footprint" "" (id 2) (at 252.73 77.47 0)
-      (effects (font (size 1.27 1.27)) hide)
-    )
-    (property "Datasheet" "https://www.usb.org/sites/default/files/documents/usb_type-c.zip" (id 3) (at 252.73 77.47 0)
-      (effects (font (size 1.27 1.27)) hide)
-    )
-    (pin "A1")
-    (pin "A10")
-    (pin "A11")
-    (pin "A12")
-    (pin "A2")
-    (pin "A3")
-    (pin "A4")
-    (pin "A5")
-    (pin "A6")
-    (pin "A7")
-    (pin "A8")
-    (pin "A9")
-    (pin "B1")
-    (pin "B10")
-    (pin "B11")
-    (pin "B12")
-    (pin "B2")
-    (pin "B3")
-    (pin "B4")
-    (pin "B5")
-    (pin "B8")
-    (pin "B9")
-    (pin "S1")
-  )
 )
